Commit message: modify URDF v

File: assets/embodiments/tianji/marvin_robot.urdf (robot description, URDF)
Before this commit: robot marvin_robot, 32 links, 31 joints
Joints:
- joint Joint1_L: limit lower=-3.1067 upper=3.1067 effort=108 velocity=0 -> lower=-3.1067 upper=3.1067 effort=108 velocity=10
- joint Joint1_R: limit lower=-3.1067 upper=3.1067 effort=108 velocity=0 -> lower=-3.1067 upper=3.1067 effort=108 velocity=10
- joint Joint2_L: limit lower=-2.0944 upper=-0.1 effort=108 velocity=0 -> lower=-2.0944 upper=-0.1 effort=108 velocity=10
- joint Joint2_R: limit lower=-2.0944 upper=-0.1 effort=108 velocity=0 -> lower=-2.0944 upper=-0.1 effort=108 velocity=10
- joint Joint3_L: limit lower=-3.1067 upper=3.1067 effort=66 velocity=0 -> lower=-3.1067 upper=3.1067 effort=66 velocity=10
- joint Joint3_R: limit lower=-3.1067 upper=3.1067 effort=66 velocity=0 -> lower=-3.1067 upper=3.1067 effort=66 velocity=10
- joint Joint4_L: limit lower=-2.5307 upper=-0.1 effort=66 velocity=0 -> lower=-2.5307 upper=-0.1 effort=66 velocity=10
- joint Joint4_R: limit lower=-2.5307 upper=-0.1 effort=66 velocity=0 -> lower=-2.5307 upper=-0.1 effort=66 velocity=10
- joint Joint5_L: limit lower=-3.1067 upper=3.1067 effort=18 velocity=0 -> lower=-3.1067 upper=3.1067 effort=18 velocity=10
- joint Joint5_R: limit lower=-3.1067 upper=3.1067 effort=18 velocity=0 -> lower=-3.1067 upper=3.1067 effort=18 velocity=10
- joint Joint6_L: limit lower=-1.0472 upper=1.0472 effort=18 velocity=0 -> lower=-1.0472 upper=1.0472 effort=18 velocity=10
- joint Joint6_R: limit lower=-1.0472 upper=1.0472 effort=18 velocity=0 -> lower=-1.0472 upper=1.0472 effort=18 velocity=10
- joint Joint7_L: limit lower=-1.5708 upper=1.5708 effort=18 velocity=0 -> lower=-1.5708 upper=1.5708 effort=18 velocity=10
- joint Joint7_R: limit lower=-1.5708 upper=1.5708 effort=18 velocity=0 -> lower=-1.5708 upper=1.5708 effort=18 velocity=10
- joint left_gripper_left_finger_joint: limit lower=0 upper=0.05 effort=30 velocity=0 -> lower=0 upper=0.05 effort=30 velocity=10
- joint left_gripper_right_finger_joint: limit lower=0 upper=0.05 effort=0 velocity=0 -> lower=0 upper=0.05 effort=0 velocity=10
- joint right_gripper_left_finger_joint: limit lower=0 upper=0.05 effort=30 velocity=0 -> lower=0 upper=0.05 effort=30 velocity=10
- joint right_gripper_right_finger_joint: limit lower=0 upper=0.05 effort=0 velocity=0 -> lower=0 upper=0.05 effort=0 velocity=10

Commit message: modify urdf

File: assets/embodiments/tianji/marvin_robot.urdf (robot description, URDF)
Before this commit: robot marvin_robot, 32 links, 31 joints
Joints:
- joint Joint1_L: limit lower=-3.1067 upper=3.1067 effort=108 velocity=10 -> lower=-3.1067 upper=3.1067 effort=108 velocity=2
- joint Joint1_R: limit lower=-3.1067 upper=3.1067 effort=108 velocity=10 -> lower=-3.1067 upper=3.1067 effort=108 velocity=2
- joint Joint2_L: limit lower=-2.0944 upper=-0.1 effort=108 velocity=10 -> lower=-2.0944 upper=-0.1 effort=108 velocity=2
- joint Joint2_R: limit lower=-2.0944 upper=-0.1 effort=108 velocity=10 -> lower=-2.0944 upper=-0.1 effort=108 velocity=2
- joint Joint3_L: limit lower=-3.1067 upper=3.1067 effort=66 velocity=10 -> lower=-3.1067 upper=3.1067 effort=66 velocity=2
- joint Joint3_R: limit lower=-3.1067 upper=3.1067 effort=66 velocity=10 -> lower=-3.1067 upper=3.1067 effort=66 velocity=2
- joint Joint4_L: limit lower=-2.5307 upper=-0.1 effort=66 velocity=10 -> lower=-2.5307 upper=-0.1 effort=66 velocity=2
- joint Joint4_R: limit lower=-2.5307 upper=-0.1 effort=66 velocity=10 -> lower=-2.5307 upper=-0.1 effort=66 velocity=2
- joint Joint5_L: limit lower=-3.1067 upper=3.1067 effort=18 velocity=10 -> lower=-3.1067 upper=3.1067 effort=18 velocity=2
- joint Joint5_R: limit lower=-3.1067 upper=3.1067 effort=18 velocity=10 -> lower=-3.1067 upper=3.1067 effort=18 velocity=2
- joint Joint6_L: limit lower=-1.0472 upper=1.0472 effort=18 velocity=10 -> lower=-1.0472 upper=1.0472 effort=18 velocity=2
- joint Joint6_R: limit lower=-1.0472 upper=1.0472 effort=18 velocity=10 -> lower=-1.0472 upper=1.0472 effort=18 velocity=2
- joint Joint7_L: limit lower=-1.5708 upper=1.5708 effort=18 velocity=10 -> lower=-1.5708 upper=1.5708 effort=18 velocity=2
- joint Joint7_R: limit lower=-1.5708 upper=1.5708 effort=18 velocity=10 -> lower=-1.5708 upper=1.5708 effort=18 velocity=2
- joint left_gripper_left_finger_joint: limit lower=0 upper=0.05 effort=30 velocity=10 -> lower=0 upper=0.05 effort=30 velocity=2
- joint left_gripper_right_finger_joint: limit lower=0 upper=0.05 effort=0 velocity=10 -> lower=0 upper=0.05 effort=0 velocity=2

Commit message: modify urdf

File: assets/embodiments/tianji/marvin_robot.urdf (robot description, URDF)
Before this commit: robot marvin_robot, 32 links, 31 joints
Joints:
- joint Joint1_L: limit lower=-3.1067 upper=3.1067 effort=108 velocity=2 -> lower=-3.1067 upper=3.1067 effort=108 velocity=10
- joint Joint1_R: limit lower=-3.1067 upper=3.1067 effort=108 velocity=2 -> lower=-3.1067 upper=3.1067 effort=108 velocity=10
- joint Joint2_L: limit lower=-2.0944 upper=-0.1 effort=108 velocity=2 -> lower=-2.0944 upper=-0.1 effort=108 velocity=10
- joint Joint2_R: limit lower=-2.0944 upper=-0.1 effort=108 velocity=2 -> lower=-2.0944 upper=-0.1 effort=108 velocity=10
- joint Joint3_L: limit lower=-3.1067 upper=3.1067 effort=66 velocity=2 -> lower=-3.1067 upper=3.1067 effort=66 velocity=10
- joint Joint3_R: limit lower=-3.1067 upper=3.1067 effort=66 velocity=2 -> lower=-3.1067 upper=3.1067 effort=66 velocity=10
- joint Joint4_L: limit lower=-2.5307 upper=-0.1 effort=66 velocity=2 -> lower=-2.5307 upper=-0.1 effort=66 velocity=10
- joint Joint4_R: limit lower=-2.5307 upper=-0.1 effort=66 velocity=2 -> lower=-2.5307 upper=-0.1 effort=66 velocity=10
- joint Joint5_L: limit lower=-3.1067 upper=3.1067 effort=18 velocity=2 -> lower=-3.1067 upper=3.1067 effort=18 velocity=10
- joint Joint5_R: limit lower=-3.1067 upper=3.1067 effort=18 velocity=2 -> lower=-3.1067 upper=3.1067 effort=18 velocity=10
- joint Joint6_L: limit lower=-1.0472 upper=1.0472 effort=18 velocity=2 -> lower=-1.0472 upper=1.0472 effort=18 velocity=10
- joint Joint6_R: limit lower=-1.0472 upper=1.0472 effort=18 velocity=2 -> lower=-1.0472 upper=1.0472 effort=18 velocity=10
- joint Joint7_L: limit lower=-1.5708 upper=1.5708 effort=18 velocity=2 -> lower=-1.5708 upper=1.5708 effort=18 velocity=10
- joint Joint7_R: limit lower=-1.5708 upper=1.5708 effort=18 velocity=2 -> lower=-1.5708 upper=1.5708 effort=18 velocity=10
- joint Link7_L_to_left_camera: origin xyz=-0.0001957 -0.2190762 0.0100948 rpy=1.532530104 1.567298900 1.543223100 -> xyz=-0.0001957 -0.2190762 0.0100948 rpy=3.103326431 1.567298900 1.543223100
- joint Link7_R_to_right_camera: origin xyz=-0.0001957 -0.2190762 0.0100948 rpy=-1.609062550 1.567298900 1.543223100 -> xyz=-0.0001957 -0.2190762 0.0100948 rpy=3.103326430 1.567298900 1.543223100
- joint left_gripper_left_finger_joint: limit lower=0 upper=0.05 effort=30 velocity=2 -> lower=0 upper=0.05 effort=30 velocity=10
- joint left_gripper_right_finger_joint: limit lower=0 upper=0.05 effort=0 velocity=2 -> lower=0 upper=0.05 effort=0 velocity=10
